File: graccel_mouse.kicad_pcb (KiCad board)
At the start: 2 copper layers, 85.9 x 67.7 mm, 41 parts, among them J1 USB_B_Micro, J2 Conn_01x08_Male, J3 Conn_01x04_Male, SW1 SW_SPDT, SW2 SW_Push, SW3 SW_Push, SW4 SW_Push, SW5 SW_Push, SW6 SW_Push, U1 AMS1117-3.3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

Commit message: complete pcb design and add gerber, bom and cpl
Parts:
- J1: footprint Connector_USB:USB_Micro-B_Wuerth_629105150521 -> Connector_USB:USB_Micro-B_Molex_47346-0001
Routing:
- net GND: track 139.0 -> 144.5 mm
- net VBUS: track 38.3 -> 39.1 mm
